File: pcb/paintable_light.kicad_sch (KiCad schematic)
At the start: 0 parts

Commit message: maybe finished schematic
Parts:
- added C1, C2, C3: 100n, Capacitor_SMD:C_0603_1608Metric_Pad1.08x0.95mm_HandSolder, symbol Device:C
- added D1, D2, D3: LED, LED_SMD:LED_0603_1608Metric_Pad1.05x0.95mm_HandSolder, symbol Device:LED
- added D4, D5, D6: LED, LED_SMD:LED_1210_3225Metric_Pad1.42x2.65mm_HandSolder, symbol Device:LED
- added J1: Conn_02x03_Counter_Clockwise, Connector_PinHeader_2.54mm:PinHeader_2x03_P2.54mm_Vertical, symbol Connector_Generic:Conn_02x03_Counter_Clockwise
- added J2: Conn_01x02, Connector_PinHeader_2.54mm:PinHeader_1x02_P2.54mm_Vertical, symbol Connector_Generic:Conn_01x02
- added R1, R4: 100, Resistor_SMD:R_0603_1608Metric_Pad0.98x0.95mm_HandSolder, symbol Device:R
- added R2, R3: 33, Resistor_SMD:R_0603_1608Metric_Pad0.98x0.95mm_HandSolder, symbol Device:R
- added R5: 10k, Resistor_SMD:R_0603_1608Metric_Pad0.98x0.95mm_HandSolder, symbol Device:R
- added U1, U2: WS2811, Package_SO:SOIC-8_3.9x4.9mm_P1.27mm, symbol Driver_LED:WS2811
- added U3: ATtiny85-20P, Package_DIP:DIP-8_W7.62mm, symbol MCU_Microchip_ATtiny:ATtiny85-20P
Connections:
- new net: D5.1 (K), U2.2 (OUTG)
- new net: D1.1 (K), U1.1 (OUTR)
- new net: D2.1 (K), U1.2 (OUTG)
- new net: C2.2, R4.2, U1.7 (SET), U1.8 (VDD)
- new net: D3.1 (K), U1.3 (OUTB)
- new net: D4.1 (K), U2.1 (OUTR)
- new net: R3.1, U1.5 (DO)
- new net: R2.1, U1.6 (DIN)
- new net: R2.2, U3.2 (XTAL1/PB3)
- new net: R3.2, U2.6 (DIN)
- new net: C1.2, R1.2, U2.7 (SET), U2.8 (VDD)
- new net: D6.1 (K), U2.3 (OUTB)
- new net +5V: C3.2, D1.2 (A), D2.2 (A), D3.2 (A), D4.2 (A), D5.2 (A), D6.2 (A), J1.6 (Pin_6), J2.1 (Pin_1), R1.1, R4.1, R5.1, U3.8 (VCC)
- new net GND: C1.1, C2.1, C3.1, J1.4 (Pin_4), J2.2 (Pin_2), U1.4 (GND), U2.4 (GND), U3.4 (GND)
- new net PROGRAM_MISO: J1.1 (Pin_1), U3.6 (PB1)
- new net PROGRAM_MOSI: J1.5 (Pin_5), U3.5 (AREF/PB0)
- new net PROGRAM_RST: J1.3 (Pin_3), R5.2, U3.1 (~{RESET}/PB5)
- new net PROGRAM_SCK: J1.2 (Pin_2), U3.7 (PB2)
- no-connect marks 0 -> 2
Other:
- note added: "Bypass capacitor"
- note added: "Bypass capacitor based on data-sheet"
- note added: "Connect SET to VDD to enable low speed mode"
- note added: "Connector for programming the MCU"
- note added: "Extra power flag after the resistor"
- note added: "LED Drivers and LEDs"
- note added: "MCU"
- note added: "Pull-up reset pin. There seems to be an internal one already which can be too weak."
- note added: "Resistor based on data-sheet"
- note added: "Resistor for impedance based on data-sheet"
- note added: "Standard Power Supply"

Commit message: initial layout
Parts:
- removed J1: Conn_02x03_Counter_Clockwise, Connector_PinHeader_2.54mm:PinHeader_2x03_P2.54mm_Vertical, symbol Connector_Generic:Conn_02x03_Counter_Clockwise
- added J3: Conn_02x03_Odd_Even, Connector_PinHeader_2.54mm:PinHeader_2x03_P2.54mm_Vertical, symbol Connector_Generic:Conn_02x03_Odd_Even
Connections:
- net +5V: now also J3.2 (Pin_2)
- net GND: now also J3.6 (Pin_6)
- net PROGRAM_MISO: now also J3.1 (Pin_1)
- net PROGRAM_MOSI: now also J3.4 (Pin_4)
- net PROGRAM_RST: now also J3.5 (Pin_5)
- net PROGRAM_SCK: now also J3.3 (Pin_3)
Changed lines of the file:
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@@
+	)
+	(symbol
+		(lib_id "Connector_Generic:Conn_02x03_Odd_Even")
+		(at 54.61 31.75 0)
+		(unit 1)
+		(exclude_from_sim no)
+		(in_bom yes)
+		(on_board yes)
+		(dnp no)
+		(fields_autoplaced yes)
+		(property "Reference" "J3"
+			(at 55.88 22.86 0)
+			(effects
+				(font
+					(size 1.27 1.27)
+				)
+			)
+		)
+		(property "Value" "Conn_02x03_Odd_Even"
+			(at 55.88 25.4 0)
+			(effects
+				(font
+					(size 1.27 1.27)
+				)
+			)
+		)
+		(property "Footprint" "Connector_PinHeader_2.54mm:PinHeader_2x03_P2.54mm_Vertical"
+			(at 54.61 31.75 0)
+			(effects
+				(font
+					(size 1.27 1.27)
+				)
+				(hide yes)
+			)
+		)
+		(property "Datasheet" "~"
+			(at 54.61 31.75 0)
+			(effects
+				(font
+					(size 1.27 1.27)
+				)
+				(hide yes)
+			)
+		)
+		(property "Description" "Generic connector, double row, 02x03, odd/even pin numbering scheme (row 1 odd numbers, row 2 even numbers), script generated (kicad-library-utils/schlib/autogen/connector/)"
+			(at 54.61 31.75 0)
+			(effects
+				(font
+					(size 1.27 1.27)
+				)
+				(hide yes)
+			)
+		)
+		(pin "6"
+		)
+		(pin "4"
+		)
+		(pin "3"
+		)
+		(pin "2"
+		)
+		(pin "1"
+		)
+		(pin "5"
+		)
+		(instances
+			(project ""
+				(path "/457c06ef-ae7c-4900-b3d7-3510fa92c411"
+					(reference "J3")
+					(unit 1)
+				)
+			)
+		)
 	)
 	(symbol
@@
 					(unit 1)
 				)
-			)
-		)
-	)
-	(symbol
-		(lib_id "Connector_Generic:Conn_02x03_Counter_Clockwise")
-		(at 54.61 31.75 0)
-		(unit 1)
-		(exclude_from_sim no)
-		(in_bom yes)
-		(on_board yes)
-		(dnp no)
-		(fields_autoplaced yes)
-		(property "Reference" "J1"
-			(at 55.88 22.86 0)
-			(effects
-				(font
-					(size 1.27 1.27)
-				)
-			)
-		)
-		(property "Value" "Conn_02x03_Counter_Clockwise"
-			(at 55.88 25.4 0)
-			(effects
-				(font
-					(size 1.27 1.27)
-				)
-			)
-		)
-		(property "Footprint" "Connector_PinHeader_2.54mm:PinHeader_2x03_P2.54mm_Vertical"
-			(at 54.61 31.75 0)
-			(effects
-				(font
-					(size 1.27 1.27)
-				)
-				(hide yes)
-			)
-		)
-		(property "Datasheet" "~"
-			(at 54.61 31.75 0)
-			(effects
-				(font
-					(size 1.27 1.27)
-				)
-				(hide yes)
-			)
-		)
-		(property "Description" "Generic connector, double row, 02x03, counter clockwise pin numbering scheme (similar to DIP package numbering), script generated (kicad-library-utils/schlib/autogen/connector/)"
-			(at 54.61 31.75 0)
-			(effects
-				(font
-					(size 1.27 1.27)
-				)
-				(hide yes)
-			)
-		)
-		(pin "2"
-		)
-		(pin "6"
-		)
-		(pin "1"
-		)
-		(pin "4"
-		)
-		(pin "3"
-		)
-		(pin "5"
-		)
-		(instances
-			(project ""
-				(path "/457c06ef-ae7c-4900-b3d7-3510fa92c411"
-					(reference "J1")
-					(unit 1)
-				)
