File: pcb/paintable_light.kicad_pcb (KiCad board)
At the start: 4 copper layers, 0 parts

Commit message: initial layout
Parts:
- added C1: 100n, Capacitor_SMD:C_0603_1608Metric_Pad1.08x0.95mm_HandSolder, F.Cu at (181.5, 53.3)
- added C2: 100n, Capacitor_SMD:C_0603_1608Metric_Pad1.08x0.95mm_HandSolder, F.Cu at (185.4, 110.6)
- added C3: 100n, Capacitor_SMD:C_0603_1608Metric_Pad1.08x0.95mm_HandSolder, F.Cu at (181.5, 58.3)
- added D1: LED, LED_SMD:LED_0603_1608Metric_Pad1.05x0.95mm_HandSolder, F.Cu at (164.8, 91.3)
- added D2: LED, LED_SMD:LED_0603_1608Metric_Pad1.05x0.95mm_HandSolder, F.Cu at (164.8, 96.0)
- added D3: LED, LED_SMD:LED_0603_1608Metric_Pad1.05x0.95mm_HandSolder, F.Cu at (164.8, 100.6)
- added D4: LED, LED_SMD:LED_1210_3225Metric_Pad1.42x2.65mm_HandSolder, F.Cu at (165.2, 108.6)
- added D5: LED, LED_SMD:LED_1210_3225Metric_Pad1.42x2.65mm_HandSolder, F.Cu at (165.2, 114.6)
- added D6: LED, LED_SMD:LED_1210_3225Metric_Pad1.42x2.65mm_HandSolder, F.Cu at (165.2, 121.3)
- added J2: Conn_01x02, Connector_PinHeader_2.54mm:PinHeader_1x02_P2.54mm_Vertical, F.Cu at (201.2, 54.3)
- added J3: Conn_02x03_Odd_Even, Connector_PinHeader_2.54mm:PinHeader_2x03_P2.54mm_Vertical, F.Cu at (196.7, 76.6)
- added R1: 100, Resistor_SMD:R_0603_1608Metric_Pad0.98x0.95mm_HandSolder, F.Cu at (181.5, 60.8)
- added R2: 33, Resistor_SMD:R_0603_1608Metric_Pad0.98x0.95mm_HandSolder, F.Cu at (170.1, 90.3)
- added R3: 33, Resistor_SMD:R_0603_1608Metric_Pad0.98x0.95mm_HandSolder, F.Cu at (180.8, 105.8)
- added R4: 100, Resistor_SMD:R_0603_1608Metric_Pad0.98x0.95mm_HandSolder, F.Cu at (185.3, 114.8)
- added R5: 10k, Resistor_SMD:R_0603_1608Metric_Pad0.98x0.95mm_HandSolder, F.Cu at (176.3, 72.6)
- added U1: WS2811, Package_SO:SOIC-8_3.9x4.9mm_P1.27mm, F.Cu at (178.5, 95.0)
- added U2: WS2811, Package_SO:SOIC-8_3.9x4.9mm_P1.27mm, F.Cu at (178.0, 115.2)
- added U3: ATtiny85-20P, Package_DIP:DIP-8_W7.62mm, F.Cu at (174.4, 77.3)

Commit message: update layout
Parts:
- D1, D2, D3, D4, D5, D6: moved to B.Cu
- moved D4 90.5 mm to (79.5, 79.5)
- moved D5 90.2 mm to (79.6, 86.2)
- moved D6 90.2 mm to (79.6, 93.0)
- moved D1 89.6 mm to (79.6, 63.8)
- moved D2 89.5 mm to (79.6, 68.8)
- moved D3 89.4 mm to (79.6, 73.8)
- moved C2 87.0 mm to (105.5, 76.0), turned to -90 degrees
- moved J2 85.0 mm to (116.2, 57.8), turned to 90 degrees
- moved C1 84.5 mm to (105.0, 89.1), turned to -90 degrees
- moved R4 83.1 mm to (110.7, 78.2), turned to 180 degrees
- moved J3 83.0 mm to (114.5, 64.7)
- moved R1 79.6 mm to (108.7, 92.9), turned to 180 degrees
- moved R5 79.5 mm to (98.3, 56.9)
- moved U2 78.2 mm to (102.5, 94.6)
- moved U1 77.4 mm to (102.5, 80.4)
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Routing:
- net Net-(D1-K): track 0.00 -> 25.7 mm, vias 0 -> 1
- net Net-(D4-K): track 0.00 -> 24.5 mm, vias 0 -> 1
- net Net-(U3-XTAL1/PB3): track 0.00 -> 24.2 mm
- net Net-(D2-K): track 0.00 -> 24.1 mm, vias 0 -> 1
- net /PROGRAM_RST: track 0.00 -> 22.9 mm
- net Net-(D3-K): track 0.00 -> 22.6 mm, vias 0 -> 1
- net Net-(D5-K): track 0.00 -> 22.1 mm, vias 0 -> 1
- net Net-(D6-K): track 0.00 -> 19.9 mm, vias 0 -> 1
- net Net-(U1-DO): track 0.00 -> 18.3 mm
- net /PROGRAM_MOSI: track 0.00 -> 13.5 mm
- net /PROGRAM_SCK: track 0.00 -> 12.8 mm
- net /PROGRAM_MISO: track 0.00 -> 8.09 mm
- net Net-(U1-SET): track 0.00 -> 7.99 mm
- net +5V: track 0.00 -> 7.38 mm, vias 0 -> 3
- net Net-(U2-SET): track 0.00 -> 6.27 mm
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- added copper zone on B.Cu, net +5V
- added copper zone on F.Cu, net GND
Other:
- board outline added: 50 x 50 mm
- board text added: "+"
- board text added: "-"
- board text added: "100nF"
- board text added: "100Ω"
- board text added: "10kΩ"
- board text added: "33Ω"
- board text added: "5V"
- board text added: "ATtiny85"
- board text added: "GND"
- board text added: "LED orientation:"
- board text added: "MISO"
- board text added: "MOSI"
- board text added: "RST"
- board text added: "SCK"
- board text added: "WS2811"
