File: pcb/paintable_light.kicad_pcb (KiCad board)
At the start: 4 copper layers, 50 x 50 mm, 19 parts, among them J2 Conn_01x02, J3 Conn_02x03_Odd_Even, U1 WS2811, U2 WS2811, U3 ATtiny85-20P

Commit message: progress
Other:
- outline, holes or cut-outs redrawn
- board text added: "Jacques Lucke Paintable Light v1 2026-02-08"
Changed lines of the file:
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@@
 		)
 	)
-	(gr_rect
-		(start 71.75 54.5)
-		(end 122.75 105.75)
-		(stroke
-			(width 0.1524)
-			(type solid)
-		)
-		(fill no)
-		(layer "B.SilkS")
-	)
-	(gr_rect
-		(start 72.25 55)
-		(end 122.25 105)
-		(stroke
-			(width 0.0381)
-			(type solid)
-		)
-		(fill no)
+	(gr_arc
+		(start 72.25 57)
+		(mid 72.835786 55.585786)
+		(end 74.25 55)
+		(stroke
+			(width 0.0381)
+			(type default)
+		)
+		(layer "Edge.Cuts")
+	)
+	(gr_arc
+		(start 122.25 103)
+		(mid 121.664214 104.414214)
+		(end 120.25 105)
+		(stroke
+			(width 0.0381)
+			(type default)
+		)
+		(layer "Edge.Cuts")
+	)
+	(gr_arc
+		(start 120.25 55)
+		(mid 121.664214 55.585786)
+		(end 122.25 57)
+		(stroke
+			(width 0.0381)
+			(type default)
+		)
+		(layer "Edge.Cuts")
+	)
+	(gr_line
+		(start 72.25 103)
+		(end 72.25 57)
+		(stroke
+			(width 0.0381)
+			(type default)
+		)
+		(layer "Edge.Cuts")
+	)
+	(gr_line
+		(start 74.25 55)
+		(end 120.25 55)
+		(stroke
+			(width 0.0381)
+			(type default)
+		)
+		(layer "Edge.Cuts")
+	)
+	(gr_line
+		(start 120.25 105)
+		(end 74.25 105)
+		(stroke
+			(width 0.0381)
+			(type default)
+		)
+		(layer "Edge.Cuts")
+	)
+	(gr_line
+		(start 122.25 57)
+		(end 122.25 103)
+		(stroke
+			(width 0.0381)
+			(type default)
+		)
+		(layer "Edge.Cuts")
+	)
+	(gr_arc
+		(start 74.25 105)
+		(mid 72.835786 104.414214)
+		(end 72.25 103)
+		(stroke
+			(width 0.0381)
+			(type default)
+		)
 		(layer "Edge.Cuts")
 	)
@@
 		(layer "F.SilkS")
 		(effects
+			(font
+				(size 0.8128 0.8128)
+				(thickness 0.1524)
+				(bold yes)
+			)
+			(justify left bottom)
+		)
+	)
+	(gr_text "Jacques Lucke\nPaintable Light v1\n2026-02-08"
+		(at 76.6 101.5 0)
+		(layer "F.SilkS")
+		(effects

Commit message: progress
Other:
- copper layers 4 -> 2
Changed lines of the file:
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@@
 	(layers
 		(0 "F.Cu" signal "Front")
-		(4 "In1.Cu" signal)
-		(6 "In2.Cu" signal)
 		(2 "B.Cu" signal "Back")
 		(13 "F.Paste" user)
@@
 			(layer "dielectric 1"
 				(type "core")
-				(thickness 0.480066)
-				(material "FR4")
-				(epsilon_r 4.5)
-				(loss_tangent 0.02)
-			)
-			(layer "In1.Cu"
-				(type "copper")
-				(thickness 0.035)
-			)
-			(layer "dielectric 2"
-				(type "prepreg")
-				(thickness 0.480066)
-				(material "FR4")
-				(epsilon_r 4.5)
-				(loss_tangent 0.02)
-			)
-			(layer "In2.Cu"
-				(type "copper")
-				(thickness 0.035)
-			)
-			(layer "dielectric 3"
-				(type "core")
-				(thickness 0.480066)
+				(thickness 1.510198)
 				(material "FR4")
 				(epsilon_r 4.5)
@@
 		(tenting front back)
 		(pcbplotparams
-			(layerselection 0x00000000_00000000_55555555_5755f5ff)
+			(layerselection 0x00000000_00000000_55555555_5755f5af)
 			(plot_on_all_layers_selection 0x00000000_00000000_00000000_00000000)
 			(disableapertmacros no)
-			(usegerberextensions no)
+			(usegerberextensions yes)
 			(usegerberattributes yes)
 			(usegerberadvancedattributes yes)
-			(creategerberjobfile yes)
+			(creategerberjobfile no)
 			(dashed_line_dash_ratio 12.000000)
 			(dashed_line_gap_ratio 3.000000)
@@
 			(outputformat 1)
 			(mirror no)
-			(drillshape 1)
+			(drillshape 0)
 			(scaleselection 1)
-			(outputdirectory "")
+			(outputdirectory "gerbers/")
 		)
 	)
