File: pcb/paintable_light.kicad_pcb (KiCad board)
At the start: 2 copper layers, 50 x 50 mm, 19 parts, among them J2 Conn_01x02, J3 Conn_02x03_Odd_Even, U1 WS2811, U2 WS2811, U3 ATtiny85-20P

Commit message: initial new board layout
Parts:
- added C4: 100n, Capacitor_SMD:C_1206_3216Metric_Pad1.33x1.80mm_HandSolder, F.Cu at (234.2, 140.5)
- added D7: LED, LED_SMD:LED_0603_1608Metric_Pad1.05x0.95mm_HandSolder, B.Cu at (236.9, 129.5)
- added D8: LED, LED_SMD:LED_0603_1608Metric_Pad1.05x0.95mm_HandSolder, B.Cu at (224.9, 136.8)
- added D9: LED, LED_SMD:LED_0603_1608Metric_Pad1.05x0.95mm_HandSolder, B.Cu at (213.1, 129.0)
- added J1: Conn_01x03_Pin, Connector_PinHeader_2.54mm:PinHeader_1x03_P2.54mm_Vertical_SMD_Pin1Left, F.Cu at (209.2, 140.5)
- added R6: 100, Resistor_SMD:R_1206_3216Metric_Pad1.30x1.75mm_HandSolder, F.Cu at (230.8, 112.9)
- added U4: CH32V003JxMx, Package_SO:JEITA_SOIC-8_3.9x4.9mm_P1.27mm, F.Cu at (240.9, 140.4)
- C1, C2, C3: footprint Capacitor_SMD:C_0603_1608Metric_Pad1.08x0.95mm_HandSolder -> Capacitor_SMD:C_1206_3216Metric_Pad1.33x1.80mm_HandSolder
- D1, D2, D3: footprint LED_SMD:LED_0603_1608Metric_Pad1.05x0.95mm_HandSolder -> LED_THT:LED_D5.0mm
- J2: value Conn_01x02 -> Conn_01x01; footprint Connector_PinHeader_2.54mm:PinHeader_1x02_P2.54mm_Vertical -> TestPoint:TestPoint_Pad_2.5x2.5mm
- J3: value Conn_02x03_Odd_Even -> Conn_01x01; footprint Connector_PinHeader_2.54mm:PinHeader_2x03_P2.54mm_Vertical -> TestPoint:TestPoint_Pad_2.5x2.5mm
- R1: value 100 -> 33; footprint Resistor_SMD:R_0603_1608Metric_Pad0.98x0.95mm_HandSolder -> Resistor_SMD:R_1206_3216Metric_Pad1.30x1.75mm_HandSolder
- R2: value 33 -> 100; footprint Resistor_SMD:R_0603_1608Metric_Pad0.98x0.95mm_HandSolder -> Resistor_SMD:R_1206_3216Metric_Pad1.30x1.75mm_HandSolder
- R3, R4: footprint Resistor_SMD:R_0603_1608Metric_Pad0.98x0.95mm_HandSolder -> Resistor_SMD:R_1206_3216Metric_Pad1.30x1.75mm_HandSolder
- R5: value 10k -> 33; footprint Resistor_SMD:R_0603_1608Metric_Pad0.98x0.95mm_HandSolder -> Resistor_SMD:R_1206_3216Metric_Pad1.30x1.75mm_HandSolder
- U3: value ATtiny85-20P -> WS2811; footprint Package_DIP:DIP-8_W7.62mm -> Package_SO:SOIC-8_3.9x4.9mm_P1.27mm
- moved D4 171.4 mm to (239.7, 140.5)
- moved D1 168.3 mm to (242.0, 108.0)
- moved D2 157.1 mm to (226.3, 125.0)
- moved D5 148.5 mm to (225.5, 114.4)
- moved R5 144.9 mm to (230.8, 115.5)
- moved U1 140.3 mm to (234.0, 129.4)
- moved R2 139.9 mm to (242.8, 128.1), turned to 180 degrees
- moved R1 139.4 mm to (242.8, 130.8), turned to 0 degrees
- moved D6 138.7 mm to (210.0, 140.5)
- moved C1 138.2 mm to (239.0, 123.1)
- moved J2 136.9 mm to (225.2, 140.5), turned to 0 degrees
- moved D3 135.1 mm to (210.3, 108.0)
- moved U3 134.1 mm to (222.3, 114.1)
- moved C3 129.7 mm to (227.2, 107.8), turned to -90 degrees
- moved J3 128.3 mm to (218.0, 140.5)
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Connections:
- C1 pad 2: Net-(U2-SET) -> Net-(U1-VDD)
- C2 pad 2: Net-(U1-SET) -> Net-(U2-VDD)
- C3 pad 2: +5V -> Net-(U3-VDD)
- J3 pad 1: /PROGRAM_MISO -> GND
- R1 pad 1: +5V -> /LED Signal
- R1 pad 2: Net-(U2-SET) -> Net-(U1-DIN)
- R2 pad 1: Net-(U1-DIN) -> +5V
- R2 pad 2: Net-(U3-XTAL1/PB3) -> Net-(U1-VDD)
- R4 pad 2: Net-(U1-SET) -> Net-(U2-VDD)
- R5 pad 1: +5V -> Net-(U2-DO)
- R5 pad 2: /PROGRAM_RST -> Net-(U3-DIN)
- U1 pad 7: Net-(U1-SET) -> unconnected-(U1-SET-Pad7)
- U1 pad 8: Net-(U1-SET) -> Net-(U1-VDD)
- U2 pad 5: unconnected-(U2-DO-Pad5) -> Net-(U2-DO)
- U2 pad 7: Net-(U2-SET) -> unconnected-(U2-SET-Pad7)
- U2 pad 8: Net-(U2-SET) -> Net-(U2-VDD)
- U3 pad 1: /PROGRAM_RST -> Net-(D7-K)
- U3 pad 2: Net-(U3-XTAL1/PB3) -> Net-(D8-K)
- U3 pad 3: unconnected-(U3-XTAL2/PB4-Pad3) -> Net-(D9-K)
- U3 pad 5: /PROGRAM_MOSI -> unconnected-(U3-DO-Pad5)
- U3 pad 6: /PROGRAM_MISO -> Net-(U3-DIN)
- U3 pad 7: /PROGRAM_SCK -> unconnected-(U3-SET-Pad7)
- U3 pad 8: +5V -> Net-(U3-VDD)
Routing:
- net Net-(D1-K): track 25.7 -> 0.00 mm, vias 1 -> 0
- net Net-(D4-K): track 24.5 -> 0.00 mm, vias 1 -> 0
- net Net-(U3-XTAL1/PB3): track 24.2 -> 0.00 mm
- net Net-(D2-K): track 24.1 -> 0.00 mm, vias 1 -> 0
- net /PROGRAM_RST: track 22.9 -> 0.00 mm
- net Net-(D3-K): track 22.6 -> 0.00 mm, vias 1 -> 0
- net Net-(D5-K): track 22.1 -> 0.00 mm, vias 1 -> 0
- net Net-(D6-K): track 19.9 -> 0.00 mm, vias 1 -> 0
- net Net-(U1-DO): track 18.3 -> 0.00 mm
- net /PROGRAM_MOSI: track 13.5 -> 0.00 mm
- net /PROGRAM_SCK: track 12.8 -> 0.00 mm
- net /PROGRAM_MISO: track 8.09 -> 0.00 mm
- net Net-(U1-SET): track 7.99 -> 0.00 mm
- net +5V: track 7.38 -> 0.00 mm, vias 3 -> 0
- net Net-(U2-SET): track 6.27 -> 0.00 mm
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- added copper zone on F.Cu, net +5V
- added copper zone on B.Cu, net GND
- removed copper zone on B.Cu, net +5V
- removed copper zone on F.Cu, net GND
Other:
- outline, holes or cut-outs redrawn
- board text removed: "+"
- board text removed: "-"
- board text removed: "100nF"
- board text removed: "100Ω"
- board text removed: "10kΩ"
- board text removed: "33Ω"
- board text removed: "5V"
- board text removed: "ATtiny85"
- board text removed: "GND"
- board text removed: "Jacques Lucke Paintable Light v1 2026-02-08"
- board text removed: "LED orientation:"
- board text removed: "MISO"
- board text removed: "MOSI"
- board text removed: "RST"
- board text removed: "SCK"
- board text removed: "WS2811"

Commit message: progress
Parts:
- moved D1 0.75 mm to (242.0, 108.8)
- moved D3 0.75 mm to (210.2, 108.8)
- moved R6 0.53 mm to (230.8, 112.3)
- moved J3 0.50 mm to (218.5, 140.5)
- moved R2 0.46 mm to (242.8, 127.6)
- moved R4 0.31 mm to (217.5, 127.5)
- turned R1 to 180 degrees
- turned R3 to 180 degrees
- turned R5 to 180 degrees
Routing:
- net /SWDIO: track 0.00 -> 49.5 mm
- net Net-(D4-K): track 0.00 -> 48.7 mm, vias 0 -> 1
- net Net-(D3-K): track 0.00 -> 37.7 mm
- net Net-(U2-DO): track 0.00 -> 34.5 mm, vias 0 -> 2
- net Net-(D5-K): track 0.00 -> 28.9 mm, vias 0 -> 1
- net Net-(D7-K): track 0.00 -> 28.9 mm, vias 0 -> 1
- net Net-(D8-K): track 0.00 -> 25.9 mm, vias 0 -> 1
- net Net-(D1-K): track 0.00 -> 23.8 mm
- net +5V: track 0.00 -> 20.6 mm, vias 0 -> 10
- net Net-(D9-K): track 0.00 -> 18.7 mm, vias 0 -> 1
- net Net-(U1-DO): track 0.00 -> 17.7 mm
- net GND: track 0.00 -> 16.0 mm, vias 0 -> 10
- net /LED Signal: track 0.00 -> 13.7 mm, vias 0 -> 2
- net Net-(D6-K): track 0.00 -> 13.5 mm, vias 0 -> 1
- net Net-(U1-VDD): track 0.00 -> 7.80 mm
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Other:
- outline, holes or cut-outs redrawn
- board text added: "+5V"
- board text added: "-+"
- board text added: "0603 LEDs"
- board text added: "100nF"
- board text added: "100Ω"
- board text added: "1210 LEDs"
- board text added: "2026-02-28"
- board text added: "33Ω"
- board text added: "Designed for"
- board text added: "GND"
- board text added: "In"
- board text added: "Jacques Lucke"
- board text added: "L"
- board text added: "M"
- board text added: "Out"
- board text added: "Paintable Light v2"
- board text added: "R"
- board text added: "SWDIO"
- board text added: "Signal"
- board text added: "THT LEDs"
- board text added: "U1 WS2811"
- board text added: "U2 WS2811"
- board text added: "U3 WS2811"
- board text added: "U4 CH32V003J4M6"

Commit message: progress
Parts:
- D1, D2, D3: footprint LED_THT:LED_D5.0mm -> front_leds:LED_1210_3225Metric_Pad1.42x2.65mm_HandSolder_front
- D4, D5, D6: footprint LED_SMD:LED_1210_3225Metric_Pad1.42x2.65mm_HandSolder -> front_leds:LED_1210_3225Metric_Pad1.42x2.65mm_HandSolder_front
- D7, D8, D9: footprint LED_SMD:LED_0603_1608Metric_Pad1.05x0.95mm_HandSolder -> front_leds:LED_1210_3225Metric_Pad1.42x2.65mm_HandSolder_front
- moved D3 38.7 mm to (224.2, 144.9), turned to -90 degrees
- moved D6 29.8 mm to (210.1, 110.7), turned to 135 degrees
- moved D4 29.7 mm to (210.1, 139.0), turned to -135 degrees
- moved D8 29.3 mm to (238.4, 110.7), turned to 45 degrees
- moved D7 27.7 mm to (224.2, 104.9), turned to 90 degrees
- moved D5 22.4 mm to (205.7, 124.9)
- moved D2 18.5 mm to (238.4, 139.0), turned to -45 degrees
- moved D1 16.3 mm to (244.2, 124.9), turned to 0 degrees
- moved D9 11.8 mm to (224.2, 124.9), turned to 0 degrees
- moved J3 10.9 mm to (229.1, 143.2)
- moved J2 4.16 mm to (229.0, 138.7)
- moved J1 1.04 mm to (209.5, 139.5)
Routing:
- net /SWDIO: track 49.5 -> 0.00 mm
- net Net-(D4-K): track 48.7 -> 0.00 mm, vias 1 -> 0
- net Net-(D3-K): track 37.7 -> 0.00 mm
- net Net-(D5-K): track 28.9 -> 0.00 mm, vias 1 -> 0
- net Net-(D7-K): track 28.9 -> 0.00 mm, vias 1 -> 0
- net Net-(D8-K): track 25.9 -> 0.00 mm, vias 1 -> 0
- net Net-(D1-K): track 23.8 -> 0.00 mm
- net +5V: track 20.6 -> 0.00 mm, vias 10 -> 0
- net Net-(D9-K): track 18.7 -> 0.00 mm, vias 1 -> 0
- net Net-(D6-K): track 13.5 -> 0.00 mm, vias 1 -> 0
- net Net-(D2-K): track 6.78 -> 0.00 mm
- net GND: track 16.0 -> 12.3 mm, vias 10 -> 8
Other:
- board text added: "1"
- board text added: "2"
- board text added: "3"
- board text added: "4"
- board text added: "5"
- board text added: "6"
- board text added: "7"
- board text added: "8"
- board text added: "9"
- board text removed: "+5V"
- board text removed: "-+"
- board text removed: "0603 LEDs"
- board text removed: "1210 LEDs"
- board text removed: "GND"
- board text removed: "L"
- board text removed: "M"
- board text removed: "R"
- board text removed: "SWDIO"
- board text removed: "THT LEDs"

Commit message: progress
Parts:
- added J4: Conn_01x01, TestPoint:TestPoint_Pad_2.5x2.5mm, F.Cu at (208.4, 140.6)
- added R7: 5k1, Resistor_SMD:R_1206_3216Metric_Pad1.30x1.75mm_HandSolder, F.Cu at (214.9, 138.6)
- added R8: 5k1, Resistor_SMD:R_1206_3216Metric_Pad1.30x1.75mm_HandSolder, F.Cu at (215.0, 142.1)
- J1: value Conn_01x03_Pin -> USB_C_Receptacle_PowerOnly_6P; footprint Connector_PinHeader_2.54mm:PinHeader_1x03_P2.54mm_Vertical_SMD_Pin1Left -> front_leds:vertical_usb_c
- moved J1 12.6 mm to (222.0, 140.8), turned to 90 degrees
- moved J2 0.10 mm to (229.1, 138.7)
Routing:
- net /SWDIO: track 0.00 -> 37.5 mm
- net Net-(D6-K): track 0.00 -> 20.2 mm, vias 0 -> 1
- net +5V: track 0.00 -> 18.9 mm, vias 0 -> 9
- net Net-(D8-K): track 0.00 -> 18.5 mm, vias 0 -> 1
- net Net-(D3-K): track 0.00 -> 17.8 mm, vias 0 -> 1
- net Net-(D4-K): track 0.00 -> 13.7 mm, vias 0 -> 1
- net Net-(D1-K): track 0.00 -> 12.9 mm, vias 0 -> 1
- net Net-(D9-K): track 0.00 -> 12.4 mm, vias 0 -> 1
- net Net-(D2-K): track 0.00 -> 12.4 mm, vias 0 -> 1
- net GND: track 12.3 -> 23.8 mm, vias 8 -> 12
- net Net-(D7-K): track 0.00 -> 7.84 mm, vias 0 -> 1
- net Net-(D5-K): track 0.00 -> 6.83 mm, vias 0 -> 1
- net Net-(J1-CC2): track 0.00 -> 5.50 mm
- net Net-(J1-CC1): track 0.00 -> 5.06 mm
Other:
- board text added: "0V"
- board text added: "2026-04-22"
- board text added: "5V"
- board text added: "GND"
- board text added: "Paintable Light v4"
- board text added: "SWDIO"
- board text removed: "2026-02-28"
- board text removed: "Paintable Light v2"

Commit message: v4
Parts:
- removed J2, J3, J4: Conn_01x01, TestPoint:TestPoint_Pad_2.5x2.5mm
- added J5: Conn_01x03_Pin, front_leds:pin_header_flat_C41417360, F.Cu at (210.4, 138.9)
- J1: footprint front_leds:vertical_usb_c -> front_leds:usb_c_vertical_C5187465
- moved J1 8.47 mm to (224.1, 132.6)
- moved R8 3.58 mm to (217.7, 139.7)
- moved R7 3.58 mm to (217.6, 136.2)
Routing:
- net Net-(J1-CC1): track 5.06 -> 9.21 mm
- net /SWDIO: track 37.5 -> 40.4 mm
- net Net-(U1-DO): track 17.7 -> 20.5 mm, vias 0 -> 2
- net Net-(J1-CC2): track 5.50 -> 6.66 mm
Other:
- board text added: "2026-05-31"
- board text removed: "2026-04-22"
